Commit message: Added Coxa and Femurs

File: src/rx1_model/urdf/rx1.urdf.xacro (robot description, xacro)
@@ -35,8 +35,34 @@
     <xacro:default_inertial mass="0.010"/>
   </link>
+  <!--**********************************************************************-->
+  <!-- Definition of the FEMUR part -->
+  <!--**********************************************************************-->
+  <xacro:macro name="femur" params="id">
+    <link name="femur_${id}">
+      <visual>
+	<origin xyz="0.075 0 -0.0146"/>
+	<geometry>
+	  <box size="0.052 0.032 0.032"/>
+	</geometry>
+	<material name="gray">
+	  <color rgba="0.4 0.4 0.4 1"/>
+	</material>
+      </visual>
+      <xacro:default_inertial mass="0.010"/>
+    </link>
+    <joint name="femur_${id}_joint" type="continuous">
+      <origin xyz="0.052 0 0" rpy="0 0 0"/>
+      <axis xyz="0 1 0"/>
+      <parent link="coxa_${id}"/>
+      <child link="femur_${id}"/>
+    </joint>
+  </xacro:macro>
+  <!--**********************************************************************-->
+  <!-- Definition of the COXA part -->
+  <!--**********************************************************************-->
   <xacro:macro name="coxa" params="id pos rot">
     <link name="coxa_${id}">
-      <origin xyz="0.026 0 0"/>
       <visual>
+	<origin xyz="0.026 0 0"/>
 	<geometry>
 	  <box size="0.052 0.048 0.025"/>
@@ -48,33 +74,17 @@
       <xacro:default_inertial mass="0.010"/>
     </link>
-    <joint name="coxa_${id}_joint" type="revolute">
-      <origin xyz="${pos}" rpy="0 0 ${rot}" />
+    <joint name="coxa_${id}_joint" type="continuous">
+      <origin xyz="${pos}" rpy="0 0 ${rot}"/>
+      <axis xyz="0 0 1"/>
       <parent link="base_link"/>
       <child link="coxa_${id}"/>
-      <limit effort="30" velocity="10" lower="${rot - 1.9}" upper="${rot + 1.9}"/>
     </joint>
+    <xacro:femur id="${id}"/>
   </xacro:macro>
   <xacro:coxa id="1" pos="0.122 0.061 -0.01375" rot="${3.14159/4}" />
   <xacro:coxa id="1R" pos="0.122 -0.061 -0.01375" rot="${-3.14159/4}" />
-  <!--**********************************************************************-->
-  <!-- Definition of the COXA part -->
-  <!--**********************************************************************-->
-  <xacro:macro name="wheel" params="number reflect">
-    <link name="coxa_${number}">
-      <visual>
-	<geometry>
-	  <cylinder radius="${wheeldiam/2}" length=".1"/>
-	</geometry>
-	<material name="black">
-	  <color rgba="0 0 0 1"/>
-	</material>
-      </visual>
-      <collision>
-	<geometry>
-	  <cylinder radius="${wheeldiam/2}" length=".1"/>
-	</geometry>
-      </collision>
-      <xacro:default_inertial mass="1"/>
-    </link>
-  </xacro:macro>
+  <xacro:coxa id="2" pos="0.0 0.1035 -0.01375" rot="${3.14159/2}" />
+  <xacro:coxa id="2R" pos="0.0 -0.1035 -0.01375" rot="${-3.14159/2}" />
+  <xacro:coxa id="3" pos="-0.122 0.061 -0.01375" rot="2.3562" />
+  <xacro:coxa id="3R" pos="-0.122 -0.061 -0.01375" rot="-2.3562" />
 </robot>

Commit message: first version (visual) of RX1

File: src/rx1_model/urdf/rx1.urdf.xacro (robot description, xacro)
@@ -22,7 +22,7 @@
     <visual>
       <geometry>
-	<box size="0.210 0.090 0.0685"/>
+	<box size="0.212 0.090 0.0685"/>
       </geometry>
-      <material name="gray">
+      <material name="gray7">
 	<color rgba="0.7 0.7 0.7 1"/>
       </material>
@@ -36,4 +36,27 @@
   </link>
   <!--**********************************************************************-->
+  <!-- Definition of the TIBIA part -->
+  <!--**********************************************************************-->
+  <xacro:macro name="tibia" params="id">
+    <link name="tibia_${id}">
+      <visual>
+	<origin xyz="0.070 0 0.0225"/>
+	<geometry>
+	  <box size="0.1 0.032 0.0125"/>
+	</geometry>
+	<material name="gray2">
+	  <color rgba="0.6 0.6 0.6 1"/>
+	</material>
+      </visual>
+      <xacro:default_inertial mass="0.010"/>
+    </link>
+    <joint name="tibia_${id}_joint" type="continuous">
+      <origin xyz="0.0644 0 -0.0146" rpy="0 ${3*pi/4} 0"/>
+      <axis xyz="0 1 0"/>
+      <parent link="femur_${id}"/>
+      <child link="tibia_${id}"/>
+    </joint>
+  </xacro:macro>
+  <!--**********************************************************************-->
   <!-- Definition of the FEMUR part -->
   <!--**********************************************************************-->
@@ -41,9 +64,9 @@
     <link name="femur_${id}">
       <visual>
-	<origin xyz="0.075 0 -0.0146"/>
+	<origin xyz="0.0384 0 0"/>
 	<geometry>
 	  <box size="0.052 0.032 0.032"/>
 	</geometry>
-	<material name="gray">
+	<material name="gray4">
 	  <color rgba="0.4 0.4 0.4 1"/>
 	</material>
@@ -52,9 +75,10 @@
     </link>
     <joint name="femur_${id}_joint" type="continuous">
-      <origin xyz="0.052 0 0" rpy="0 0 0"/>
+      <origin xyz="0.052 0 0" rpy="0 ${-pi/4} 0"/>
       <axis xyz="0 1 0"/>
       <parent link="coxa_${id}"/>
       <child link="femur_${id}"/>
     </joint>
+    <xacro:tibia id="${id}"/>
   </xacro:macro>
   <!--**********************************************************************-->
@@ -68,5 +92,5 @@
 	  <box size="0.052 0.048 0.025"/>
 	</geometry>
-	<material name="gray">
+	<material name="gray5">
 	  <color rgba="0.5 0.5 0.5 1"/>
 	</material>
@@ -82,4 +106,43 @@
     <xacro:femur id="${id}"/>
   </xacro:macro>
+  <!--**********************************************************************-->
+  <!-- Definition of the HEAD -->
+  <!--**********************************************************************-->
+  <link name="head_pivot">
+    <visual>
+      <origin xyz="0.00125 0 0"/>
+      <geometry>
+	<box size="0.048 0.038 0.038"/>
+      </geometry>
+      <material name="red6">
+	<color rgba="0.7 0.6 0.6 1"/>
+      </material>
+    </visual>
+    <xacro:default_inertial mass="0.010"/>
+  </link>
+  <joint name="head_pivot_joint" type="continuous">
+    <origin xyz="${0.106+0.0455} 0 0.00525" rpy="0 0 0.5"/>
+    <axis xyz="0 0 1"/>
+    <parent link="base_link"/>
+    <child link="head_pivot"/>
+  </joint>
+  <link name="camera_head">
+    <visual>
+      <origin xyz="0.042 0 0"/>
+      <geometry>
+	<box size="0.018 0.016 0.016"/>
+      </geometry>
+      <material name="blue1">
+	<color rgba="0.5 0.5 0.99 1"/>
+      </material>
+    </visual>
+    <xacro:default_inertial mass="0.010"/>
+  </link>
+  <joint name="head_tilt_joint" type="continuous">
+    <origin xyz="0.0133 0 0.004" rpy="0 0 0"/>
+    <axis xyz="0 0 1"/>
+    <parent link="head_pivot"/>
+    <child link="camera_head"/>
+  </joint>
   <xacro:coxa id="1" pos="0.122 0.061 -0.01375" rot="${3.14159/4}" />
   <xacro:coxa id="1R" pos="0.122 -0.061 -0.01375" rot="${-3.14159/4}" />
